File: kicad/simple-dock/simple-dock.kicad_pcb (KiCad board)
At the start: 2 copper layers, 89.1 x 95.3 mm, 64 parts, among them J1 Conn_02x40_Odd_Even, J18 HDMI_A, J2 Conn_02x06_Odd_Even, J23 line, J3 Micro_SD_Card_Det2, Q1 A03400, Q2 A03400, Q3 A03400, U29 PT8211, U32 LM324A

Commit message: more kicad
Parts:
- added J4: Conn_02x20_Odd_Even, Connector_PinHeader_2.54mm:PinHeader_2x20_P2.54mm_Vertical_SMD, F.Cu at (67.9, 57.6)
- added U22: generic_2048x8_TSOP_II_44_BB, Package_SO:TSSOP-44_4.4x11mm_P0.5mm, F.Cu at (43.2, 38.7)
- added U23: generic_2048x8_TSOP_II_44, Package_SO:TSSOP-44_4.4x11mm_P0.5mm, F.Cu at (52.3, 38.7)
Connections:
- C2399 pad 10: /SOM_FPGA/B2_D19 -> /SOM_FPGA/A0
- C2399 pad 11: /SOM_FPGA/B2_A20 -> /SOM_FPGA/D11
- C2399 pad 12: /SOM_FPGA/B2_E19 -> /SOM_FPGA/A1
- C2399 pad 13: /SOM_FPGA/B2_B20 -> /SOM_FPGA/D10
- C2399 pad 16: /SOM_FPGA/B2_C19 -> /SOM_FPGA/A2
- C2399 pad 17: /SOM_FPGA/B2_A19 -> /SOM_FPGA/A7
- C2399 pad 18: /SOM_FPGA/B2_C18 -> /SOM_FPGA/A3
- C2399 pad 19: /SOM_FPGA/B2_A18 -> /SOM_FPGA/A8
- C2399 pad 22: /SOM_FPGA/B1_E17 -> /SOM_FPGA/~{CAS}
- C2399 pad 23: /SOM_FPGA/B2_B18 -> /SOM_FPGA/A12
- C2399 pad 24: /SOM_FPGA/B1_F16 -> /SOM_FPGA/~{RAS}
- C2399 pad 25: /SOM_FPGA/B2_B17 -> /SOM_FPGA/CLK
- C2399 pad 28: /SOM_FPGA/B1_D16 -> /SOM_FPGA/~{WE}
- C2399 pad 29: /SOM_FPGA/B2_C17 -> /SOM_FPGA/A9
- C2399 pad 30: /SOM_FPGA/B1_E16 -> /SOM_FPGA/A4
- C2399 pad 31: /SOM_FPGA/B2_D17 -> /SOM_FPGA/A11
- C2399 pad 34: /SOM_FPGA/B1_D15 -> /SOM_FPGA/A5
- C2399 pad 35: /SOM_FPGA/B2_A16 -> /SOM_FPGA/D13
- C2399 pad 36: /SOM_FPGA/B1_D14 -> /SOM_FPGA/A6
- C2399 pad 37: /SOM_FPGA/B2_A15 -> /SOM_FPGA/D12
- C2399 pad 4: /SOM_FPGA/B2_C20 -> /SOM_FPGA/BA1
- C2399 pad 40: /SOM_FPGA/B1_F15 -> /SOM_FPGA/BA0
- C2399 pad 41: /SOM_FPGA/B2_B16 -> /SOM_FPGA/D15
- C2399 pad 42: /SOM_FPGA/B1_F14 -> /SOM_FPGA/LDM
- C2399 pad 43: /SOM_FPGA/B2_B15 -> /SOM_FPGA/D14
- C2399 pad 44: /SOM_FPGA/B1_F13 -> /SOM_FPGA/UDM
- C2399 pad 47: /SOM_FPGA/B2_A14 -> /SOM_FPGA/D6
- C2399 pad 49: /SOM_FPGA/B2_A13 -> /SOM_FPGA/D7
- C2399 pad 5: /SOM_FPGA/B2_A21 -> /SOM_FPGA/D9
- C2399 pad 53: /SOM_FPGA/B2_B13 -> /SOM_FPGA/D4
- C2399 pad 55: /SOM_FPGA/B2_C13 -> /SOM_FPGA/D5
- C2399 pad 59: /SOM_FPGA/B2_C15 -> /SOM_FPGA/D2
- C2399 pad 6: /SOM_FPGA/B2_D20 -> /SOM_FPGA/A10
- C2399 pad 61: /SOM_FPGA/B2_C14 -> /SOM_FPGA/D3
- C2399 pad 65: /SOM_FPGA/B2_E14 -> /SOM_FPGA/D0
- C2399 pad 67: /SOM_FPGA/B2_E13 -> /SOM_FPGA/D1
- C2399 pad 7: /SOM_FPGA/B2_B21 -> /SOM_FPGA/D8
- C2399 pad 78: unconnected-(C2399-Pin_78-Pad78) -> /SOM_FPGA/Q0_LN2_RX.N
- C2399 pad 80: unconnected-(C2399-Pin_80-Pad80) -> /SOM_FPGA/Q0_LN2_RX.P
- J1 pad 72: /SOM_FPGA/B2_F21 -> /SOM_FPGA/~{CS}
- U29 pad 4: GNDAudio -> GND
