File: kicad/simple-dock/SOM_FPGA.kicad_sch (KiCad schematic)
At the start: 3 parts, among them J1 Conn_02x40_Odd_Even

Commit message: more kicad
Connections:
- net B4_G15 renamed DVI_CK.P
- net B4_G16 renamed DVI_CK.N
- net B4_H14 renamed DVI_D0.N
- net B4_H15 renamed DVI_D1.N
- net B4_J14 renamed DVI_D0.P
- net B4_J15 renamed DVI_D1.P
- net B4_K13 renamed DVI_HPD
- net B4_K14 renamed DVI_PWR
- net B5_J17 renamed DVI_D2.N
- net B5_K17 renamed DVI_D2.P
- net B5_L13 renamed EDID_SDA
- net B5_M13 renamed EDID_SCL
- net B6_U15 renamed DBUG.TX
- net B6_V15 renamed SDIO.CLK
- net B7_AA15 renamed SDIO.D0
- net B7_AA16 renamed DAT
- net B7_AB17 renamed WS
- net B7_W15 renamed SDIO.D3
- net B7_Y16 renamed SDIO.CMD
- net B7_Y17 renamed BCK
- net B8_AB15 renamed SDIO.D1
- net B8_W14 renamed SDIO.D2
- net B9_Y13 renamed SDIO.DET
- net JTAG_TCK renamed JTAG.TCK
- net JTAG_TDI renamed JTAG.TDI
- net JTAG_TDO renamed JTAG.TDO
- net JTAG_TMS renamed JTAG.TMS
- net MODE0 renamed MODE.0
- net MODE1 renamed MODE.1
- net MODE2 renamed MODE.2
Other:
- note added: "B4_G15"
- note added: "B4_G16"
- note added: "B4_H14"
- note added: "B4_H15"
- note added: "B4_J14"
- note added: "B4_J15"
- note added: "B4_K13"
- note added: "B4_K14"
- note added: "B5_J17"
- note added: "B5_K17"
- note added: "B5_L13"
- note added: "B5_M13"
- note added: "B6_U15"
- note added: "B6_V15"
- note added: "B7_AA15"
- note added: "B7_AA16"
- note added: "B7_AB17"
- note added: "B7_W15"
- note added: "B7_Y16"
- note added: "B7_Y17"
- note added: "B8_AB15"
- note added: "B8_W14"
- note added: "B9_Y13"

Commit message: more kicad
Parts:
- C2399, C2400: footprint (none) -> Connector_Hirose_DF40:Hirose_DF40HC(3.0)-100DS-0.4V_2x50_P0.4mm
- J1: footprint (none) -> Connector_Hirose_DF40:Hirose_DF40HC(3.0)-80DS-0.4V_2x40_P0.4mm
Changed lines of the file:
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@@
 			)
 		)
-		(property "Footprint" ""
+		(property "Footprint" "Connector_Hirose_DF40:Hirose_DF40HC(3.0)-100DS-0.4V_2x50_P0.4mm"
 			(at 153.67 78.74 0)
 			(effects
@@
 			)
 		)
-		(property "Footprint" ""
+		(property "Footprint" "Connector_Hirose_DF40:Hirose_DF40HC(3.0)-80DS-0.4V_2x40_P0.4mm"
 			(at 233.68 80.01 0)
 			(effects
@@
 			)
 		)
-		(property "Footprint" ""
+		(property "Footprint" "Connector_Hirose_DF40:Hirose_DF40HC(3.0)-100DS-0.4V_2x50_P0.4mm"
 			(at 58.42 76.2 0)
 			(effects

Commit message: more kicad
Connections:
- net Q0_LN2_RX.N: now also C2399.78 (Pin_78)
- net Q0_LN2_RX.P: now also C2399.80 (Pin_80)
- net B1_D14 renamed A6
- net B1_D15 renamed A5
- net B1_D16 renamed ~{WE}
- net B1_E16 renamed A4
- net B1_E17 renamed ~{CAS}
- net B1_F13 renamed UDM
- net B1_F14 renamed LDM
- net B1_F15 renamed BA0
- net B1_F16 renamed ~{RAS}
- net B2_A13 renamed D7
- net B2_A14 renamed D6
- net B2_A15 renamed D12
- net B2_A16 renamed D13
- net B2_A18 renamed A8
- net B2_A19 renamed A7
- net B2_A20 renamed D11
- net B2_A21 renamed D9
- net B2_B13 renamed D4
- net B2_B15 renamed D14
- net B2_B16 renamed D15
- net B2_B17 renamed CLK
- net B2_B18 renamed A12
- net B2_B20 renamed D10
- net B2_B21 renamed D8
- net B2_C13 renamed D5
- net B2_C14 renamed D3
- net B2_C15 renamed D2
- net B2_C17 renamed A9
- net B2_C18 renamed A3
- net B2_C19 renamed A2
- net B2_C20 renamed BA1
- net B2_D17 renamed A11
- net B2_D19 renamed A0
- net B2_D20 renamed A10
- net B2_E13 renamed D1
- net B2_E14 renamed D0
- net B2_E19 renamed A1
- net B2_F21 renamed ~{CS}
- net B8_V14 renamed DBUG.RX
Other:
- note added: "B1_D14"
- note added: "B1_D15"
- note added: "B1_D16"
- note added: "B1_E16"
- note added: "B1_E17"
- note added: "B1_F13"
- note added: "B1_F14"
- note added: "B1_F15"
- note added: "B1_F16"
- note added: "B2_A13"
- note added: "B2_A14"
- note added: "B2_A15"
- note added: "B2_A16"
- note added: "B2_A18"
- note added: "B2_A19"
- note added: "B2_A20"
- note added: "B2_A21"
- note added: "B2_B13"
- note added: "B2_B15"
- note added: "B2_B16"
- note added: "B2_B17"
- note added: "B2_B18"
- note added: "B2_B20"
- note added: "B2_B21"
- note added: "B2_C13"
- note added: "B2_C14"
- note added: "B2_C15"
- note added: "B2_C17"
- note added: "B2_C18"
- note added: "B2_C19"
- note added: "B2_C20"
- note added: "B2_D17"
- note added: "B2_D19"
- note added: "B2_D20"
- note added: "B2_E13"
- note added: "B2_E14"
- note added: "B2_E19"
- note added: "B2_F21"
- note added: "B8_V14"

Commit message: more kicad
Connections:
- net B5_M15 is gone; now on net D.P: C2400.18 (Pin_18)
- net B5_M16 is gone; now on net D.N: C2400.16 (Pin_16)
- net B4_G13 renamed D.N
- net B4_H13 renamed D.P
Other:
- note added: "B4_G13"
- note added: "B4_H13"
- note added: "B5_M15"
- note added: "B5_M16"
Changed lines of the file:
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@@
 		)
 	)
+	(bus_alias "USBA1"
+		(members "D.N" "D.P")
+	)
+	(bus_alias "USBA2"
+		(members "D.N" "D.P")
+	)
 	(text "B12_U13_TDO"
 		(exclude_from_sim no)
@@
 		)
 	)
+	(text "B4_G13"
+		(exclude_from_sim no)
+		(at 76.2 109.22 0)
+		(effects
+			(font
+				(size 1.27 1.27)
+			)
+			(justify right bottom)
+		)
+	)
 	(text "B2_A14"
 		(exclude_from_sim no)
@@
 		)
 	)
+	(text "B5_M16"
+		(exclude_from_sim no)
+		(at 168.91 48.26 0)
+		(effects
+			(font
+				(size 1.27 1.27)
+			)
+			(justify right bottom)
+		)
+	)
 	(text "B8_V14"
 		(exclude_from_sim no)
@@
 		)
 	)
+	(text "B4_H13"
+		(exclude_from_sim no)
+		(at 76.2 111.76 0)
+		(effects
+			(font
+				(size 1.27 1.27)
+			)
+			(justify right bottom)
+		)
+	)
 	(text "B4_G16"
 		(exclude_from_sim no)
@@
 		)
 	)
+	(text "B5_M15"
+		(exclude_from_sim no)
+		(at 168.91 50.8 0)
+		(effects
+			(font
+				(size 1.27 1.27)
+			)
+			(justify right bottom)
+		)
+	)
 	(text "B9_Y13"
 		(exclude_from_sim no)
@@
 	)
 	(bus_entry
+		(at 90.17 109.22)
+		(size 2.54 2.54)
+		(stroke
+			(width 0)
+			(type default)
+		)
+	)
+	(bus_entry
 		(at 185.42 66.04)
 		(size 2.54 2.54)
@@
 	)
 	(bus_entry
+		(at 185.42 50.8)
+		(size 2.54 2.54)
+		(stroke
+			(width 0)
+			(type default)
+		)
+	)
+	(bus_entry
 		(at 26.67 30.48)
 		(size 2.54 2.54)
@@
 	)
 	(bus_entry
+		(at 185.42 48.26)
+		(size 2.54 2.54)
+		(stroke
+			(width 0)
+			(type default)
+		)
+	)
+	(bus_entry
 		(at 90.17 101.6)
 		(size 2.54 2.54)
@@
 	)
 	(bus_entry
+		(at 90.17 111.76)
+		(size 2.54 2.54)
+		(stroke
+			(width 0)
+			(type default)
+		)
+	)
+	(bus_entry
 		(at 90.17 106.68)
 		(size 2.54 2.54)
@@
 	(bus
 		(pts
+			(xy 187.96 50.8) (xy 187.96 53.34)
+		)
+		(stroke
+			(width 0)
+			(type default)
+		)
+	)
+	(bus
+		(pts
 			(xy 121.92 109.22) (xy 121.92 111.76)
 		)
@@
 		)
 	)
+	(bus
+		(pts
+			(xy 187.96 53.34) (xy 189.23 53.34)
+		)
+		(stroke
+			(width 0)
+			(type default)
+		)
+	)
 	(wire
 		(pts
@@
 		)
 	)
+	(bus
+		(pts
+			(xy 92.71 111.76) (xy 92.71 114.3)
+		)
+		(stroke
+			(width 0)
+			(type default)
+		)
+	)
 	(wire
 		(pts
@@
 		)
 	)
+	(bus
+		(pts
+			(xy 92.71 114.3) (xy 93.98 114.3)
+		)
+		(stroke
+			(width 0)
+			(type default)
+		)
+	)
 	(wire
 		(pts
@@
 	(bus
 		(pts
-			(xy 116.84 113.03) (xy 121.92 113.03)
+			(xy 120.65 113.03) (xy 121.92 113.03)
 		)
 		(stroke
@@
 		)
 	)
+	(label "D.N"
+		(at 185.42 48.26 180)
+		(effects
+			(font
+				(size 1.27 1.27)
+			)
+			(justify right bottom)
+		)
+	)
 	(label "B3_N12_NRECONFIG"
 		(at 204.47 107.95 0)
@@
 		)
 	)
+	(label "D.N"
+		(at 90.17 109.22 180)
+		(effects
+			(font
+				(size 1.27 1.27)
+			)
+			(justify right bottom)
+		)
+	)
 	(label "Q0_LN2_RX.P"
 		(at 90.17 127 180)
@@
 		)
 	)
-	(label "B4_G13"
-		(at 90.17 109.22 180)
-		(effects
-			(font
-				(size 1.27 1.27)
-			)
-			(justify right bottom)
-		)
-	)
 	(label "B5_G20"
 		(at 265.43 110.49 180)
@@
 		)
 	)
-	(label "B5_M15"
-		(at 185.42 50.8 180)
-		(effects
-			(font
-				(size 1.27 1.27)
-			)
-			(justify right bottom)
-		)
-	)
 	(label "Q0_LN1_TX.P"
 		(at 29.21 149.86 0)
@@
 		)
 	)
+	(label "D.P"
+		(at 185.42 50.8 180)
+		(effects
+			(font
+				(size 1.27 1.27)
+			)
+			(justify right bottom)
+		)
+	)
 	(label "SDIO.CMD"
 		(at 185.42 81.28 180)
@@
 		)
 	)
-	(label "B5_M16"
-		(at 185.42 48.26 180)
-		(effects
-			(font
-				(size 1.27 1.27)
-			)
-			(justify right bottom)
-		)
-	)
 	(label "B7_U21"
 		(at 204.47 46.99 0)
@@
 		)
 	)
+	(label "D.P"
+		(at 90.17 111.76 180)
+		(effects
+			(font
+				(size 1.27 1.27)
+			)
+			(justify right bottom)
+		)
+	)
 	(label "JTAG.TMS"
 		(at 205.74 34.29 0)
@@
 		)
 	)
-	(label "B4_H13"
-		(at 90.17 111.76 180)
-		(effects
-			(font
-				(size 1.27 1.27)
-			)
-			(justify right bottom)
-		)
-	)
 	(hierarchical_label "{DVI}"
 		(shape bidirectional)
@@
 		)
 	)
+	(hierarchical_label "{USBA1}"
+		(shape bidirectional)
+		(at 189.23 53.34 0)
+		(effects
+			(font
+				(size 1.27 1.27)
+			)
+			(justify left)
+		)
+	)
 	(hierarchical_label "MODE{0 1 2}"
 		(shape input)
-		(at 116.84 113.03 180)
+		(at 120.65 113.03 180)
 		(effects
 			(font
@@
 		(effects
 			(font
+				(size 1.27 1.27)
+			)
+			(justify left)
+		)
+	)
+	(hierarchical_label "{USBA2}"
+		(shape bidirectional)
+		(at 93.98 114.3 0)
+		(effects
+			(font
