File: kicad/simple-dock/_autosave-simple-dock.kicad_pcb (KiCad board)
At the start: 2 copper layers, 89.1 x 95.3 mm, 73 parts, among them J1 Conn_02x40_Odd_Even, J18 HDMI_A, J2 Conn_02x06_Odd_Even, J23 line, J3 Micro_SD_Card_Det2, J4 Conn_02x20_Odd_Even, Q1 A03400, Q2 A03400, Q3 A03400, U1 24AA64-I_OT, U22 generic_2048x8_TSOP_II_44_BB, U23 generic_2048x8_TSOP_II_44, U29 PT8211, U32 LM324A, U6 74LS00_FULL

Commit message: more kicad
Parts:
- added REF**: MountingHole_2.2mm_M2_DIN965, MountingHole:MountingHole_2.2mm_M2_DIN965, F.Cu at (123.0, 52.0)
- added REF**: MountingHole_2.2mm_M2_DIN965, MountingHole:MountingHole_2.2mm_M2_DIN965, F.Cu at (82.0, 83.0)
- added REF**: MountingHole_2.2mm_M2_DIN965, MountingHole:MountingHole_2.2mm_M2_DIN965, F.Cu at (123.0, 83.0)
- added REF**: MountingHole_2.2mm_M2_DIN965, MountingHole:MountingHole_2.2mm_M2_DIN965, F.Cu at (82.0, 52.0)
