File: kicad/simple-dock/jtag_debug.kicad_sch (KiCad schematic)
At the start: 1 part, among them J2 Conn_02x06_Odd_Even

Commit message: more kicad
Parts:
- J2: footprint (none) -> Connector_PinSocket_2.54mm:PinSocket_2x06_P2.54mm_Horizontal
Changed lines of the file:
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@@
 			)
 		)
-		(property "Footprint" ""
+		(property "Footprint" "Connector_PinSocket_2.54mm:PinSocket_2x06_P2.54mm_Horizontal"
 			(at 105.41 57.15 0)
 			(effects
