File: kicad/simple-dock/sdcard.kicad_sch (KiCad schematic)
At the start: 8 parts, among them J3 Micro_SD_Card_Det2

Commit message: more kicad
Parts:
- J3: footprint (none) -> mod:hirose_micro_sd_card_socket
Changed lines of the file:
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@@
 			)
 		)
-		(property "Footprint" ""
+		(property "Footprint" "mod:hirose_micro_sd_card_socket"
 			(at 196.85 58.42 0)
 			(effects
