File: kicad/simple-dock/sdram.kicad_sch (KiCad schematic)
At the start: 9 parts, among them J4 Conn_02x20_Odd_Even, U1 24AA64-I_OT, U22 generic_2048x8_TSOP_II_44_BB, U23 generic_2048x8_TSOP_II_44, U6 74LS00_FULL

Commit message: more kicad
Parts:
- U22, U23: footprint Package_SO:TSSOP-44_4.4x11mm_P0.5mm -> Package_SO:TSOP-II-44_10.16x18.41mm_P0.8mm
Changed lines of the file:
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@@
 			)
 		)
-		(property "Footprint" "Package_SO:TSSOP-44_4.4x11mm_P0.5mm"
+		(property "Footprint" "Package_SO:TSOP-II-44_10.16x18.41mm_P0.8mm"
 			(at 217.17 46.99 0)
 			(effects
@@
 			)
 		)
-		(property "Footprint" "Package_SO:TSSOP-44_4.4x11mm_P0.5mm"
+		(property "Footprint" "Package_SO:TSOP-II-44_10.16x18.41mm_P0.8mm"
 			(at 151.13 46.99 0)
 			(effects
